Commit message: before flexbe

File: src/aubo_ros2_driver/aubo_description/urdf/scene.xacro (robot description, xacro)
@@ -1,4 +1,8 @@
 <?xml version="1.0"?>
-<robot xmlns:xacro="http://ros.org/wiki/xacro">
+<robot xmlns:xacro="http://www.ros.org/wiki/xacro">
+  <!-- Определяем цвет -->
+  <material name="gray">
+    <color rgba="0.5 0.5 0.5 1.0"/>
+  </material>
   <!-- Стол -->
   <link name="table">
@@ -19,17 +23,15 @@
       <mass value="50"/>
       <origin xyz="0 0 0"/>
-      <inertia
-          ixx="1"
-          ixy="0"
-          ixz="0"
-          iyy="1"
-          iyz="0"
-          izz="1"/>
+      <inertia ixx="1" ixy="0" ixz="0" iyy="1" iyz="0" izz="1"/>
     </inertial>
   </link>
   <joint name="table_joint" type="fixed">
-      <parent link="world"/>
-      <child link="table"/>
-      <origin xyz="0 0 0"/>
+    <parent link="world"/>
+    <child link="table"/>
+    <origin xyz="0 0 0"/>
   </joint>
+  <!-- Цвет стола в самом Gazebo (Gazebo игнорирует material из visual) -->
+  <gazebo reference="table">
+    <material>Gazebo/Grey</material>
+  </gazebo>
 </robot>

File: src/aubo_ros2_driver/aubo_description/urdf/xacro/inc/aubo_gazebo.xacro (robot description, xacro)
@@ -8,4 +8,6 @@
     transmission_hw_interface="$(arg transmission_hw_interface)"
     aubo_type="${aubo_type}"/>
+    <!-- Подключаем сцену (стол) -->
+  <xacro:include filename="$(find aubo_description)/urdf/scene.xacro"/>
   <ros2_control name="auboGazeboSystem" type="system">
     <hardware>

Commit message: FlexBE: behavior test7 (joint-space move via MoveIt) + правки launch/xacro

File: src/aubo_ros2_driver/aubo_description/urdf/scene.xacro (robot description, xacro)
@@ -1,22 +1,28 @@
 <?xml version="1.0"?>
 <robot xmlns:xacro="http://www.ros.org/wiki/xacro">
-  <!-- Определяем цвет -->
   <material name="gray">
     <color rgba="0.5 0.5 0.5 1.0"/>
   </material>
-  <!-- Стол -->
+  <material name="red">
+    <color rgba="0.8 0.1 0.1 1.0"/>
+  </material>
+  <material name="green">
+    <color rgba="0.1 0.7 0.1 1.0"/>
+  </material>
+  <material name="blue">
+    <color rgba="0.1 0.3 0.8 1.0"/>
+  </material>
+  <!-- ===================== СТОЛ ===================== -->
+  <!-- Верхняя грань на z = -0.02 (на 2 см НИЖЕ основания робота),
+       чтобы база не продавливала столешницу. -->
   <link name="table">
     <visual>
-      <origin xyz="0.6 0.0 -0.05"/>
-      <geometry>
-        <box size="1.0 1.0 0.1"/>
-      </geometry>
+      <origin xyz="0 0 0"/>
+      <geometry><box size="1.0 1.0 0.1"/></geometry>
       <material name="gray"/>
     </visual>
     <collision>
-      <origin xyz="0.6 0.0 -0.05"/>
-      <geometry>
-        <box size="1.0 1.0 0.1"/>
-      </geometry>
+      <origin xyz="0 0 0"/>
+      <geometry><box size="1.0 1.0 0.1"/></geometry>
     </collision>
     <inertial>
@@ -27,11 +33,90 @@
   </link>
   <joint name="table_joint" type="fixed">
-    <parent link="world"/>
+    <parent link="base_link"/>
     <child link="table"/>
-    <origin xyz="0 0 0"/>
+    <origin xyz="0 0 -0.07" rpy="0 0 0"/>
   </joint>
-  <!-- Цвет стола в самом Gazebo (Gazebo игнорирует material из visual) -->
   <gazebo reference="table">
     <material>Gazebo/Grey</material>
+    <selfCollide>false</selfCollide>
+    <maxContacts>0</maxContacts>
+  </gazebo>
+  <!-- ===================== КУБИКИ ===================== -->
+  <!-- Стоят на столешнице (её верх z=-0.02), центр куба z = -0.02 + 0.025 = 0.005.
+       Отодвинуты дальше от базы робота, чтобы не мешать первым звеньям. -->
+  <link name="cube_red">
+    <visual>
+      <origin xyz="0 0 0"/>
+      <geometry><box size="0.05 0.05 0.05"/></geometry>
+      <material name="red"/>
+    </visual>
+    <collision>
+      <origin xyz="0 0 0"/>
+      <geometry><box size="0.05 0.05 0.05"/></geometry>
+    </collision>
+    <inertial>
+      <mass value="0.2"/>
+      <inertia ixx="0.0001" ixy="0" ixz="0" iyy="0.0001" iyz="0" izz="0.0001"/>
+    </inertial>
+  </link>
+  <joint name="cube_red_joint" type="fixed">
+    <parent link="base_link"/>
+    <child link="cube_red"/>
+    <origin xyz="0.45 0.25 0.005" rpy="0 0 0"/>
+  </joint>
+  <gazebo reference="cube_red">
+    <material>Gazebo/Red</material>
+    <selfCollide>false</selfCollide>
+    <maxContacts>0</maxContacts>
+  </gazebo>
+  <link name="cube_green">
+    <visual>
+      <origin xyz="0 0 0"/>
+      <geometry><box size="0.05 0.05 0.05"/></geometry>
+      <material name="green"/>
+    </visual>
+    <collision>
+      <origin xyz="0 0 0"/>
+      <geometry><box size="0.05 0.05 0.05"/></geometry>
+    </collision>
+    <inertial>
+      <mass value="0.2"/>
+      <inertia ixx="0.0001" ixy="0" ixz="0" iyy="0.0001" iyz="0" izz="0.0001"/>
+    </inertial>
+  </link>
+  <joint name="cube_green_joint" type="fixed">
+    <parent link="base_link"/>
+    <child link="cube_green"/>
+    <origin xyz="0.45 -0.25 0.005" rpy="0 0 0"/>
+  </joint>
+  <gazebo reference="cube_green">
+    <material>Gazebo/Green</material>
+    <selfCollide>false</selfCollide>
+    <maxContacts>0</maxContacts>
+  </gazebo>
+  <link name="cube_blue">
+    <visual>
+      <origin xyz="0 0 0"/>
+      <geometry><box size="0.05 0.05 0.05"/></geometry>
+      <material name="blue"/>
+    </visual>
+    <collision>
+      <origin xyz="0 0 0"/>
+      <geometry><box size="0.05 0.05 0.05"/></geometry>
+    </collision>
+    <inertial>
+      <mass value="0.2"/>
+      <inertia ixx="0.0001" ixy="0" ixz="0" iyy="0.0001" iyz="0" izz="0.0001"/>
+    </inertial>
+  </link>
+  <joint name="cube_blue_joint" type="fixed">
+    <parent link="base_link"/>
+    <child link="cube_blue"/>
+    <origin xyz="0.55 0.0 0.005" rpy="0 0 0"/>
+  </joint>
+  <gazebo reference="cube_blue">
+    <material>Gazebo/Blue</material>
+    <selfCollide>false</selfCollide>
+    <maxContacts>0</maxContacts>
   </gazebo>
 </robot>

File: src/aubo_ros2_driver/aubo_description/urdf/xacro/inc/aubo_gazebo.xacro (robot description, xacro)
@@ -8,6 +8,71 @@
     transmission_hw_interface="$(arg transmission_hw_interface)"
     aubo_type="${aubo_type}"/>
-    <!-- Подключаем сцену (стол) -->
-  <xacro:include filename="$(find aubo_description)/urdf/scene.xacro"/>
+  <joint name="world_to_table" type="fixed">
+      <parent link="world"/>
+      <child link="table"/>
+      <origin xyz="0 0 -0.7" rpy="0 0 0"/>
+    </joint>
+  <link name="table">
+    <visual>
+      <origin xyz="0 0 0.35" rpy="0 0 0"/>
+      <geometry>
+        <box size="1.2 0.8 0.7"/>
+      </geometry>
+      <material name="table_wood">
+        <color rgba="0.6 0.45 0.3 1.0"/>
+      </material>
+    </visual>
+    <collision>
+      <origin xyz="0 0 0.35" rpy="0 0 0"/>
+      <geometry>
+        <box size="1.2 0.8 0.7"/>
+      </geometry>
+    </collision>
+    <inertial>
+      <origin xyz="0 0 0.35" rpy="0 0 0"/>
+      <mass value="50.0"/>
+      <inertia ixx="5.0" ixy="0.0" ixz="0.0" iyy="7.0" iyz="0.0" izz="8.0"/>
+    </inertial>
+  </link>
+  <xacro:macro name="scene_cube" params="name x y z r g b">
+    <joint name="world_to_${name}" type="fixed">
+      <parent link="world"/>
+      <child link="${name}"/>
+      <origin xyz="${x} ${y} ${z}" rpy="0 0 0"/>
+    </joint>
+    <link name="${name}">
+      <visual>
+        <origin xyz="0 0 0" rpy="0 0 0"/>
+        <geometry>
+          <box size="0.05 0.05 0.05"/>
+        </geometry>
+        <material name="mat_${name}">
+          <color rgba="${r} ${g} ${b} 1.0"/>
+        </material>
+      </visual>
+      <collision>
+        <origin xyz="0 0 0" rpy="0 0 0"/>
+        <geometry>
+          <box size="0.05 0.05 0.05"/>
+        </geometry>
+      </collision>
+      <inertial>
+        <origin xyz="0 0 0" rpy="0 0 0"/>
+        <mass value="0.2"/>
+        <inertia ixx="0.0001" ixy="0.0" ixz="0.0" iyy="0.0001" iyz="0.0" izz="0.0001"/>
+      </inertial>
+    </link>
+    <gazebo reference="${name}">
+      <material>Gazebo/Grey</material>
+      <selfCollide>false</selfCollide>
+    </gazebo>
+  </xacro:macro>
+  <xacro:scene_cube name="cube_red"   x="0.45" y="0.15"  z="0.025" r="0.9" g="0.1" b="0.1"/>
+  <xacro:scene_cube name="cube_green" x="0.45" y="0.0"   z="0.025" r="0.1" g="0.8" b="0.1"/>
+  <xacro:scene_cube name="cube_blue"  x="0.45" y="-0.15" z="0.025" r="0.1" g="0.2" b="0.9"/>
+  <gazebo reference="table">
+    <material>Gazebo/Wood</material>
+    <selfCollide>false</selfCollide>
+  </gazebo>
   <ros2_control name="auboGazeboSystem" type="system">
     <hardware>
@@ -18,4 +83,5 @@
       <state_interface name="position"><param name="initial_value">0.0</param></state_interface>
       <state_interface name="velocity"/>
+      <state_interface name="effort"/>
     </joint>
     <joint name="upperArm_joint">
@@ -23,4 +89,5 @@
       <state_interface name="position"><param name="initial_value">0.0</param></state_interface>
       <state_interface name="velocity"/>
+      <state_interface name="effort"/>
     </joint>
     <joint name="foreArm_joint">
@@ -28,4 +95,5 @@
       <state_interface name="position"><param name="initial_value">0.0</param></state_interface>
       <state_interface name="velocity"/>
+      <state_interface name="effort"/>
     </joint>
     <joint name="wrist1_joint">
@@ -33,4 +101,5 @@
       <state_interface name="position"><param name="initial_value">0.0</param></state_interface>
       <state_interface name="velocity"/>
+      <state_interface name="effort"/>
     </joint>
     <joint name="wrist2_joint">
@@ -38,4 +107,5 @@
       <state_interface name="position"><param name="initial_value">0.0</param></state_interface>
       <state_interface name="velocity"/>
+      <state_interface name="effort"/>
     </joint>
     <joint name="wrist3_joint">
@@ -43,8 +113,12 @@
       <state_interface name="position"><param name="initial_value">0.0</param></state_interface>
       <state_interface name="velocity"/>
+      <state_interface name="effort"/>
     </joint>
   </ros2_control>
   <gazebo>
     <plugin filename="libgazebo_ros2_control.so" name="gazebo_ros2_control">
+      <robot_param>robot_description</robot_param>
+      <robot_param_node>robot_state_publisher</robot_param_node>
+      <controller_manager_name>controller_manager</controller_manager_name>
       <parameters>$(find aubo_gazebo)/config/aubo_controllers.yaml</parameters>
     </plugin>

File: src/aubo_ros2_driver/aubo_description/urdf/xacro/inc/aubo_ros2_macro.xacro (robot description, xacro)
@@ -1,97 +1,43 @@
 <?xml version="1.0"?>
 <robot xmlns:xacro="http://ros.org/wiki/xacro">
-  <xacro:macro name="aubo_robot" params="aubo_type transmission_hw_interface">
-    <xacro:include filename="$(find aubo_description)/urdf/${aubo_type}.urdf.xacro" />
-    <joint name="ee_fixed_joint" type="fixed">
-      <parent link="wrist3_Link" />
-      <child link ="ee_link" />
-      <origin xyz="0.0 0.0 0.0" rpy="0.0 0.0 ${pi/2.0}" />
-    </joint>
-    <link name="ee_link">
-      <collision>
-        <geometry>
-          <box size="0.01 0.01 0.01"/>
-        </geometry>
-        <origin rpy="0 0 0" xyz="-0.01 0 0"/>
-      </collision>
-    </link>
-    <transmission name="shoulder_trans">
-      <type>transmission_interface/SimpleTransmission</type>
-      <joint name="shoulder_joint">
-        <hardwareInterface>${transmission_hw_interface}</hardwareInterface>
-      </joint>
-      <actuator name="shoulder_motor">
-        <mechanicalReduction>1</mechanicalReduction>
-      </actuator>
-    </transmission>
-    <transmission name="foreArm_trans">
-      <type>transmission_interface/SimpleTransmission</type>
-      <joint name="foreArm_joint">
-        <hardwareInterface>${transmission_hw_interface}</hardwareInterface>
-      </joint>
-      <actuator name="foreArm_motor">
-        <mechanicalReduction>1</mechanicalReduction>
-      </actuator>
-    </transmission>
-    <transmission name="upperArm_trans">
-      <type>transmission_interface/SimpleTransmission</type>
-      <joint name="upperArm_joint">
-        <hardwareInterface>${transmission_hw_interface}</hardwareInterface>
-      </joint>
-      <actuator name="upperArm_motor">
-        <mechanicalReduction>1</mechanicalReduction>
-      </actuator>
-    </transmission>
-    <transmission name="wrist1_trans">
-      <type>transmission_interface/SimpleTransmission</type>
-      <joint name="wrist1_joint">
-        <hardwareInterface>${transmission_hw_interface}</hardwareInterface>
-      </joint>
-      <actuator name="wrist1_motor">
-        <mechanicalReduction>1</mechanicalReduction>
-      </actuator>
-    </transmission>
-    <transmission name="wrist2_trans">
-      <type>transmission_interface/SimpleTransmission</type>
-      <joint name="wrist2_joint">
-        <hardwareInterface>${transmission_hw_interface}</hardwareInterface>
-      </joint>
-      <actuator name="wrist2_motor">
-        <mechanicalReduction>1</mechanicalReduction>
-      </actuator>
-    </transmission>
-    <transmission name="wrist3_trans">
-      <type>transmission_interface/SimpleTransmission</type>
-      <joint name="wrist3_joint">
-        <hardwareInterface>${transmission_hw_interface}</hardwareInterface>
-      </joint>
-      <actuator name="wrist3_motor">
-        <mechanicalReduction>1</mechanicalReduction>
-      </actuator>
-    </transmission>
-    <gazebo reference="shoulder_Link">
-      <selfCollide>true</selfCollide>
-    </gazebo>
-    <gazebo reference="upperArm_Link">
-      <selfCollide>true</selfCollide>
-    </gazebo>
-    <gazebo reference="foreArm_Link">
-      <selfCollide>true</selfCollide>
-    </gazebo>
-    <gazebo reference="wrist1_Link">
-      <selfCollide>true</selfCollide>
-    </gazebo>
-    <gazebo reference="wrist2_Link">
-      <selfCollide>true</selfCollide>
-    </gazebo>
-    <gazebo reference="wrist3_Link">
-      <selfCollide>true</selfCollide>
-    </gazebo>
-    <gazebo reference="ee_link">
-      <selfCollide>true</selfCollide>
-    </gazebo>
-    <gazebo>
-      <!-- plugin name="ros_control" filename="libgazebo_ros_control.so"/ -->
-    </gazebo>
-  </xacro:macro>
+<xacro:macro name="aubo_robot" params="aubo_type transmission_hw_interface">
+<xacro:include filename="$(find aubo_description)/urdf/${aubo_type}.urdf.xacro" />
+<joint name="ee_fixed_joint" type="fixed">
+<parent link="wrist3_Link" />
+<child link ="ee_link" />
+<origin xyz="0.0 0.0 0.0" rpy="0.0 0.0 ${pi/2.0}" />
+</joint>
+<link name="ee_link">
+<collision>
+<geometry>
+<box size="0.01 0.01 0.01"/>
+</geometry>
+<origin rpy="0 0 0" xyz="-0.01 0 0"/>
+</collision>
+</link>
+<gazebo reference="base_link">
+<selfCollide>false</selfCollide>
+</gazebo>
+<gazebo reference="shoulder_Link">
+<selfCollide>false</selfCollide>
+</gazebo>
+<gazebo reference="upperArm_Link">
+<selfCollide>false</selfCollide>
+</gazebo>
+<gazebo reference="foreArm_Link">
+<selfCollide>false</selfCollide>
+</gazebo>
+<gazebo reference="wrist1_Link">
+<selfCollide>false</selfCollide>
+</gazebo>
+<gazebo reference="wrist2_Link">
+<selfCollide>false</selfCollide>
+</gazebo>
+<gazebo reference="wrist3_Link">
+<selfCollide>false</selfCollide>
+</gazebo>
+<gazebo reference="ee_link">
+<selfCollide>false</selfCollide>
+</gazebo>
+</xacro:macro>
 </robot>
