Commit message: FlexBE: joint-space + Cartesian motions working

File: src/aubo_ros2_driver/aubo_description/urdf/xacro/inc/aubo_gazebo.xacro (robot description, xacro)
@@ -47,5 +47,5 @@
           <box size="0.05 0.05 0.05"/>
         </geometry>
-        <material name="mat_${name}">
+        <material name="${name}_material">
           <color rgba="${r} ${g} ${b} 1.0"/>
         </material>
